File: RF Signal Strength Circuit/RF Circuit/RF Circuit.kicad_sch (KiCad schematic)
At the start: 0 parts

Commit message: Updated folders
Parts:
- added C1, C21, C3: 22uF/10V(20%), symbol Device:C
- added C14, C19, C9: 0.1uF/50V(10%), symbol Device:C
- added C20: 10uF/10V(20%), symbol Device:C
- added C22: 0.1uF/50v(10%), symbol Device:C
- added D1: SFH4346(RED LED), LED_THT:LED_D3.0mm_IRBlack, symbol LED:SFH4346
- added D3: BAT760-7, Diode_THT:D_DO-35_SOD27_P7.62mm_Horizontal, symbol Diode:BAT85
- added D4, D5, D6: LESD5D5.0CI1G, symbol Device:D_TVS
- added J1: USB_B_Micro, symbol Connector:USB_B_Micro
- added Q1, Q2: SS8050, Package_TO_SOT_SMD:SOT-23, symbol Transistor_BJT:SS8050
- added R11: 10K(5%), symbol Device:R_Small_US
- added R17, R18: 0R(5%), symbol Device:R_US
- added R2: 2k(5%), symbol Device:R_US
- added R21, R22: 10k(5%), symbol Device:R_US
- added R24: 2k(5%), symbol Device:R_Small_US
- added R25: 22.1k(1%), symbol Device:R_Small_US
- added R26: 47.5k(1%), symbol Device:R_Small_US
- added SW1, SW2: SW_Push, symbol Switch:SW_Push
- added U1: ESP32-WROOM-32E, RF_Module:ESP32-WROOM-32E, symbol RF_Module:ESP32-WROOM-32E
- added U2: CP2102N-A02-GQFN28, easyeda2kicad:QFN-28_L5.0-W5.0-P0.50-TL-EP3.3, symbol easyeda2kicad:CP2102N-A02-GQFN28
- added U3: AMS1117-3.3, Package_TO_SOT_SMD:SOT-223-3_TabPin2, symbol Regulator_Linear:AMS1117-3.3
Connections:
- new net: D1.2 (A), R2.2
- new net: R24.1, U2.9 (RSTb)
- new net: Q1.1 (B), R21.2
- new net: R25.2, R26.2, U2.8 (VBUS)
- new net: Q2.1 (B), R22.2
- new net ACTIVE: U2.11 (SUSPENDb)
- new net CTS: U2.23 (CTS)
- new net D+: D4.2 (A2), J1.3 (D+), U2.4 (D+)
- new net D-: D5.2 (A2), J1.2 (D-), U2.5 (D-)
- new net DCD: U2.1 (DCD)
- new net DSR: U2.27 (DSR)
- new net DTR: Q2.2 (E), R21.1, U2.28 (DTR)
- new net EN: C14.2, C9.1, Q1.3 (C), R11.2, SW2.2, U1.3 (EN)
- new net EXT_5V: C1.1, D3.1 (K), R2.1, U3.3 (VI)
- new net GND: C1.2, C14.1, C19.2, C20.2, C21.2, C22.2, C3.2, C9.2, D1.1 (K), D4.1 (A1), D5.1 (A1), D6.1 (A1), J1.5 (GND), J1.SH (Shield), R26.1, SW1.1, SW2.1, U1.[1,15,38,39] (GND), U2.29 (EP), U2.3 (GND), U3.1 (GND)
- new net IO0: Q2.3 (C), SW1.2, U1.25 (IO0)
- new net IO12: U1.14 (IO12)
- new net IO13: U1.16 (IO13)
- new net IO14: U1.13 (IO14)
- new net IO15: U1.23 (IO15)
- new net IO16: U1.27 (IO16)
- new net IO17: U1.28 (IO17)
- new net IO18: U1.30 (IO18)
- new net IO19: U1.31 (IO19)
- new net IO2: U1.24 (IO2)
- new net IO21: U1.33 (IO21)
- new net IO22: U1.36 (IO22)
- new net IO23: U1.37 (IO23)
- new net IO25: U1.10 (IO25)
- new net IO26: U1.11 (IO26)
- new net IO27: U1.12 (IO27)
- new net IO32: U1.8 (IO32)
- new net IO33: U1.9 (IO33)
- new net IO34: U1.6 (IO34)
- new net IO35: U1.7 (IO35)
- new net IO4: U1.26 (IO4)
- new net IO5: U1.29 (IO5)
- new net RI: U2.2 (RI/CLK)
- new net RTS: Q1.2 (E), R22.1, U2.24 (RTS)
- new net RXD: R17.2, U2.25 (RXD)
- new net RXD0: R18.1, U1.34 (RXD0/IO3)
- new net SENSOR_VN: U1.5 (SENSOR_VN)
- new net SENSOR_VP: U1.4 (SENSOR_VP)
- new net TXD: R18.2, U2.26 (TXD)
- new net TXD0: R17.1, U1.35 (TXD0/IO1)
- new net VBUS: D3.2 (A), D6.2 (A2), J1.1 (VBUS), R25.1
- new net VDD33: C19.1, C20.1, C21.1, C22.1, C3.1, R11.1, R24.2, U1.2 (VDD), U2.6 (VDD), U2.7 (VREGIN), U3.2 (VO)
- no-connect marks 0 -> 13
Other:
- note added: "Auto program DTR RTS --> EN 1O0 1 1 1 1 0 0 1 1 1 0 0 1 0 1 1 0"
- note added: "ESP32 Module"
- note added: "Micro USB 5V&USB-UART"
- note added: "Power Supply"
- note added: "Schematics: https://dl.espressif.com/dl/schematics/esp32_devkitc_v4_sch.pdf"
- note added: "Switch Button"

Commit message: Updates on schematics / imported symbols and footprints
Parts:
- added BT1: Lipo Battery, symbol Device:Battery_Cell
- added D2: D_Schottky, symbol Device:D_Schottky
- added SW3: SW_SPST, symbol Switch:SW_SPST
Connections:
- net EXT_5V: now also D2.1 (K)
- net GND: now also BT1.2 (-)
- new net: BT1.1 (+), SW3.1 (A)
- new net: D2.2 (A), SW3.2 (B)
Other:
- added sheet RF Connections (untitled.kicad_sch)
- note added: "Antenna Selection: https://www.johansontechnology.com/docs/4470/johanson-antenna-selection-guide_YA3dQmX.pdf(Chose 915MHz)"
- note added: "Battery Voltage has to be in specific range"
- note added: "Chosen Antenna: https://www.johansontechnology.com/products/antennas/rf-antennas/0915at43a0026001e/"
- note added: "ESP-32 Schematic: https://dl.espressif.com/dl/schematics/esp32_devkitc_v4_sch.pdf"
- note added: "Transcevier Datasheet: https://www.semtech.com/products/wireless-rf/frequency-shift-keying-fsk/sx1211"
- note removed: "Schematics: https://dl.espressif.com/dl/schematics/esp32_devkitc_v4_sch.pdf"
- moved on the sheet: C1, C14, C21, C22, C3, C9, D1, R11, R2, SW1, SW2, U1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

Commit message: First finished schematic
Parts:
- added J2: SSD1306, symbol Connector:Conn_01x04_Pin
Connections:
- net GND: now also J2.GND (Pin_1)
- net VDD33: now also J2.VCC33 (Pin_2)
- net IO18 renamed SCK
- net IO19 renamed MISO
- net IO21 renamed SDA
- net SDA: now also J2.SDA (Pin_4)
- net IO22 renamed SCL
- net SCL: now also J2.SCL (Pin_3)
- net IO23 renamed MOSI
- net IO25 renamed IRQ_1
- net IO27 renamed IRQ_0
- net IO33 renamed PLL_LOCK
- net IO5 renamed NSS_CONFIG
Other:
- note added: "Display Module"
- note added: "ESP-32 Datasheet: https://documentation.espressif.com/esp32-wroom-32e_esp32-wroom-32ue_datasheet_en.html#[11,%22XYZ%22,56.69,711.37,null]"
- note removed: "Antenna Selection: https://www.johansontechnology.com/docs/4470/johanson-antenna-selection-guide_YA3dQmX.pdf(Chose 915MHz)"
- note removed: "Chosen Antenna: https://www.johansontechnology.com/products/antennas/rf-antennas/0915at43a0026001e/"
- note removed: "Transcevier Datasheet: https://www.semtech.com/products/wireless-rf/frequency-shift-keying-fsk/sx1211"
