File: RF Signal Strength Circuit/RF Circuit/untitled.kicad_sch (KiCad schematic)
At the start: 15 parts, among them U5 SX1211I084TRT

Commit message: First finished schematic
Parts:
- added C1, C2: 1uF(15%), symbol Device:C
- added C3: 220nF(10%), symbol Device:C
- added C5: 100nF(10%), symbol Device:C
- added C6: 10nF(10%), symbol Device:C
- added C7: 680pF(5%), symbol Device:C
- added L1: 8.2nH(+-0.2nH), symbol Device:L
- added L2: 6.8nH(+-0.2nH), symbol Device:L
- added Q1: ABM3B-155-12.800MHZ-T, C1985396:CRYSTAL-SMD_4P-L5.0-W3.2-BL, symbol C1985396:ABM3B-155-12.800MHZ-T
- added R2: 6.8kΩ(1%), symbol Device:R_US
Connections:
- net GND: now also U5.1 (TEST5), U5.12 (TEST0), U5.2 (TEST1), U5.30 (TEST4), U5.32 (NC), U5.8 (TEST6), U5.9 (TEST7), C1.2, C5.1, Q1.2 (GND), Q1.4 (GND)
- net at U5.10 (XTAL_P): now also Q1.1
- net at U5.11 (XTAL_M): now also Q1.3
- net NSS_CONFIG: now reaches U5.14 (NSS_CONFIG)
- net NSS_DATA: now reaches U5.15 (NSS_DATA)
- net MISO: now reaches U5.16 (MISO)
- net MOSI: now reaches U5.17 (MOSI)
- net SCK: now reaches U5.18 (SCK)
- net IRQ_0: now reaches U5.21 (IRQ_0)
- net IRQ_1: now reaches U5.22 (IRQ_1)
- net PLL_LOCK: now reaches U5.23 (PLL_LOCK)
- net VDD33: now reaches U5.26 (VDD)
- net VDD33: now also C1.1
- net at U5.27 (VR_1V): now also C2.1
- net at U5.28 (VR_DIG): now also C3.1
- net at U5.3 (VR_VCO): now also C5.2, L1.1, L2.1
- net at U5.4 (VCO_M): now also L1.2
- net at U5.5 (VCO_P): now also L2.2
- net at U5.6 (LF_M): now also C6.2, C7.1
- net at U5.7 (LF_P): now also C7.2, R2.1
- new net: C6.1, R2.2
- no-connect marks 0 -> 3
Other:
- note added: "Antenna Selection: https://www.johansontechnology.com/docs/4470/johanson-antenna-selection-guide_YA3dQmX.pdf(Chose 915MHz)"
- note added: "Chosen Antenna: https://www.johansontechnology.com/products/antennas/rf-antennas/0915at43a0026001e/"
- note added: "May need to add parallel capacitors"
- note added: "Transcevier Datasheet: https://www.semtech.com/products/wireless-rf/frequency-shift-keying-fsk/sx1211"
- moved on the sheet: AE2, C11, C12(NC), C18, C4, C50, C51, C8, C9, L3, L4, L49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
